File: RP2024_Module34/RP2024_Module34.kicad_pcb (KiCad board)
At the start: 2 copper layers, 34.5 x 49 mm, 47 parts, among them J1 USB_C_Receptacle_USB2.0, J3 Conn_02x15_Odd_Even, U1 XC6206PxxxMR-Regulator_Linear, U2 PRTR5V0U2X, U3 W25Q128JVS, U4 RP2040, U5 74LVC1T45, Y1 12Mhz

Commit message: Add files via upload
Parts:
- removed REF** (x3): MountingHole_2.2mm_M2, MountingHole:MountingHole_2.2mm_M2
- J3: value Conn_02x15_Odd_Even -> Conn_02x17_Odd_Even; footprint MyConnectors:IDC_2X15_1.27MM -> MyConnectors:IDC_2X17_1.27MM
- moved J3 2.56 mm to (141.0, 104.3)
Connections:
- J3 pad 10: RGB_DATA -> R_A
- J3 pad 11: COL4 -> COL2
- J3 pad 12: ROW5 -> Caps
- J3 pad 13: COL5 -> COL3
- J3 pad 14: ROW4 -> RGB_DATA
- J3 pad 15: COL6 -> COL4
- J3 pad 16: ROW3 -> ROW5
- J3 pad 17: COL7 -> COL5
- J3 pad 18: ROW2 -> ROW4
- J3 pad 19: COL8 -> COL6
- J3 pad 20: ROW1 -> ROW3
- J3 pad 21: COL9 -> COL7
- J3 pad 22: ROW0 -> ROW2
- J3 pad 23: COL10 -> COL8
- J3 pad 24: COL17 -> ROW1
- J3 pad 25: COL11 -> COL9
- J3 pad 26: COL16 -> ROW0
- J3 pad 27: COL12 -> COL10
- J3 pad 28: COL15 -> COL17
- J3 pad 29: COL13 -> COL11
- J3 pad 3: COL0 -> GND
- J3 pad 30: COL14 -> COL16
- J3 pad 4: R_B -> VBUS
- J3 pad 5: COL1 -> unconnected-(J3-Pin_5-Pad5)
- J3 pad 6: R_A -> Scroll
- J3 pad 7: COL2 -> COL0
- J3 pad 8: Caps -> R_B
- J3 pad 9: COL3 -> COL1
Routing:
- net VBUS: track 85.2 -> 115.7 mm, vias 5 -> 7
- net RGB_DATA: track 63.4 -> 60.2 mm
- net GND: track 106.4 -> 108.1 mm
- net Caps: track 46.9 -> 46.3 mm
Other:
- board text added: "ScLk"
