File: 34 Pin Extender Board/adapter64.kicad_pcb (KiCad board)
At the start: 2 copper layers, 35 x 57 mm, 5 parts, among them J5 Conn_01x21_Pin, J6 Conn_02x17_Odd_Even, J7 Conn_01x21_Pin

Commit message: Add files via upload
Updates
Other:
- board text added: "Keyboard Module Expander Version 2.0 D"
- board text added: "Keyboard Module Expander Version 2.0D"
